File: Tap_Photosensor_PCB.kicad_pcb (KiCad board)
At the start: 2 copper layers, 28.8 x 14.3 mm, 14 parts, among them J1 Conn_01x03, U1 L78L05_SOT89, U3 ITR9608

Commit message: Adding panelization and R3
Parts:
- removed the REF** at (107.4, 62.2)
- removed the REF** at (109.6, 67.4)
- added R1: 1k, Resistor_SMD:R_0603_1608Metric, F.Cu at (111.2, 66.9)
- R3: value 640R -> 500R
Connections:
- R3 pad 1: +5V -> Net-(U3-Emitter)
- U3 pad 4: GND -> Net-(U3-Emitter)
Routing:
- net Net-(U3-Emitter): track 0.00 -> 7.64 mm
- net +5V: track 0.00 -> 7.48 mm
- net SIG: track 8.33 -> 11.7 mm
- net GND: vias 14 -> 6
Other:
- board text added: "rev BEANS 3"
- board text removed: "rev BEANS 2"

Commit message: fixing mistake
Parts:
- removed the REF** at (122.6, 61.0)
Connections:
- R1 pad 2: SIG -> Net-(U3-Collector)
- R3 pad 1: Net-(U3-Emitter) -> SIG
- U3 pad 3: SIG -> Net-(U3-Collector)
- U3 pad 4: Net-(U3-Emitter) -> SIG
Routing:
- net Net-(U3-Emitter): track 7.64 -> 0.00 mm
- net Net-(U3-Collector): track 0.00 -> 2.88 mm
- net SIG: track 11.7 -> 12.5 mm
Changed lines of the file:
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@@
 	(net 5 "/current limit u3 led")
 	(net 6 "/current limit status led")
-	(net 7 "Net-(U3-Emitter)")
+	(net 7 "Net-(U3-Collector)")
 	(footprint "Diode_SMD:D_SOD-123"
 		(layer "F.Cu")
@@
 			(layers "F.Cu" "F.Mask" "F.Paste")
 			(roundrect_rratio 0.25)
-			(net 1 "SIG")
+			(net 7 "Net-(U3-Collector)")
 			(pintype "passive")
 		)
@@
 			(layers "*.Cu" "*.Mask")
 			(remove_unused_layers no)
-			(net 1 "SIG")
+			(net 7 "Net-(U3-Collector)")
 			(pinfunction "Collector")
 			(pintype "open_collector")
@@
 			(layers "*.Cu" "*.Mask")
 			(remove_unused_layers no)
-			(net 7 "Net-(U3-Emitter)")
+			(net 1 "SIG")
 			(pinfunction "Emitter")
 			(pintype "output")
@@
 			(layers "F.Cu" "F.Mask" "F.Paste")
 			(roundrect_rratio 0.25)
-			(net 7 "Net-(U3-Emitter)")
+			(net 1 "SIG")
 			(pintype "passive")
 		)
@@
 		(embedded_fonts no)
 	)
-	(footprint "Fiducial:Fiducial_0.5mm_Mask1mm"
-		(layer "F.Cu")
-		(at 122.6 61)
-		(descr "Circular Fiducial, 0.5mm bare copper, 1mm soldermask opening (Level C)")
-		(tags "fiducial")
-		(property "Reference" "REF**"
-			(at 0 -1.5 0)
-			(layer "F.SilkS")
-			(hide yes)
-			(effects
-				(font
-					(size 1 1)
-					(thickness 0.15)
-				)
-			)
-		)
-		(property "Value" "Fiducial_0.5mm_Mask1mm"
-			(at 0 1.5 0)
-			(layer "F.Fab")
-			(hide yes)
-			(effects
-				(font
-					(size 1 1)
-					(thickness 0.15)
-				)
-			)
-		)
-		(property "Datasheet" ""
-			(at 0 0 0)
-			(layer "F.Fab")
-			(hide yes)
-			(effects
-				(font
-					(size 1.27 1.27)
-					(thickness 0.15)
-				)
-			)
-		)
-		(property "Description" ""
-			(at 0 0 0)
-			(layer "F.Fab")
-			(hide yes)
-			(effects
-				(font
-					(size 1.27 1.27)
-					(thickness 0.15)
-				)
-			)
-		)
-		(attr smd)
-		(fp_circle
-			(center 0 0)
-			(end 0.75 0)
-			(stroke
-				(width 0.05)
-				(type solid)
-			)
-			(fill no)
-			(layer "F.CrtYd")
-		)
-		(fp_circle
-			(center 0 0)
-			(end 0.5 0)
-			(stroke
-				(width 0.1)
-				(type solid)
-			)
-			(fill no)
-			(layer "F.Fab")
-		)
-		(fp_text user "${REFERENCE}"
-			(at 0 0 0)
-			(layer "F.Fab")
-			(effects
-				(font
-					(size 0.2 0.2)
-					(thickness 0.04)
-				)
-			)
-		)
-		(pad "" smd circle
-			(at 0 0)
-			(size 0.5 0.5)
-			(layers "F.Cu" "F.Mask")
-			(solder_mask_margin 0.25)
-			(clearance 0.25)
-		)
-		(embedded_fonts no)
-	)
 	(footprint "MountingHole:MountingHole_3.2mm_M3_ISO7380"
 		(layer "F.Cu")
@@
 	)
 	(segment
+		(start 107.58 61.42)
+		(end 107.58 64.42)
+		(width 0.25)
+		(layer "F.Cu")
+		(net 1)
+	)
+	(segment
 		(start 108.2 60.8)
 		(end 109.2 60.8)
@@
 	)
 	(segment
-		(start 107.52 66.9)
-		(end 107.5 66.92)
+		(start 111.69125 64.42)
+		(end 114.18625 61.925)
 		(width 0.25)
 		(layer "F.Cu")
@@
 	)
 	(segment
-		(start 110.375 66.9)
-		(end 107.52 66.9)
+		(start 107.58 64.42)
+		(end 111.69125 64.42)
 		(width 0.25)
 		(layer "F.Cu")
@@
 	)
 	(segment
-		(start 105.8 63.2)
-		(end 108.2 60.8)
-		(width 0.25)
-		(layer "F.Cu")
-		(net 1)
-	)
-	(segment
-		(start 105.8 65.22)
-		(end 105.8 63.2)
-		(width 0.25)
-		(layer "F.Cu")
-		(net 1)
-	)
-	(segment
-		(start 107.5 66.92)
-		(end 105.8 65.22)
+		(start 108.2 60.8)
+		(end 107.58 61.42)
 		(width 0.25)
 		(layer "F.Cu")
@@
 	)
 	(segment
-		(start 111.69125 64.42)
-		(end 114.18625 61.925)
+		(start 107.52 66.9)
+		(end 107.5 66.92)
 		(width 0.25)
 		(layer "F.Cu")
@@
 	)
 	(segment
-		(start 107.58 64.42)
-		(end 111.69125 64.42)
+		(start 110.375 66.9)
+		(end 107.52 66.9)
 		(width 0.25)
 		(layer "F.Cu")
