File: panel/Tap_photosensor_PCB.kicad_pcb (KiCad board)
At the start: 2 copper layers, 152.1 x 159.3 mm, 659 parts, among them J1 Conn_01x03, U1 L78L05_SOT89, U3 ITR9608

Commit message: updating panel
Parts:
- removed the REF** at (189.6, 91.9)
- removed the REF** at (127.9, 48.9)
- removed the REF** at (158.7, 48.9)
- removed the REF** at (97.1, 134.9)
- removed the REF** at (127.9, 91.9)
- removed the REF** at (97.1, 63.2)
- removed the REF** at (97.1, 77.6)
- removed the REF** at (127.9, 120.5)
- removed the REF** at (189.6, 48.9)
- removed the REF** at (189.6, 149.2)
- removed the REF** at (220.4, 34.6)
- removed the REF** at (189.6, 120.5)
- removed the REF** at (220.4, 149.2)
- removed the REF** at (158.7, 163.5)
- removed the REF** at (97.1, 106.2)
- removed the REF** at (220.4, 48.9)
- removed the REF** at (97.1, 48.9)
- removed the REF** at (97.1, 120.5)
- removed the REF** at (158.7, 106.2)
- removed the REF** at (97.1, 149.2)
- removed the REF** at (127.9, 77.6)
- removed the REF** at (189.6, 63.2)
- removed the REF** at (220.4, 163.5)
- removed the REF** at (127.9, 134.9)
- removed the REF** at (158.7, 63.2)
- removed the REF** at (158.7, 134.9)
- removed the REF** at (158.7, 91.9)
- removed the REF** at (97.1, 34.6)
- removed the REF** at (127.9, 34.6)
- removed the REF** at (220.4, 91.9)
- removed the REF** at (127.9, 149.2)
- removed the REF** at (189.6, 77.6)
- removed the REF** at (189.6, 134.9)
- removed the REF** at (158.7, 34.6)
- removed the REF** at (97.1, 163.5)
- removed the REF** at (220.4, 134.9)
- removed the REF** at (189.6, 106.2)
- removed the REF** at (189.6, 163.5)
- removed the REF** at (158.7, 77.6)
- removed the REF** at (220.4, 120.5)
- removed the REF** at (97.1, 91.9)
- removed the REF** at (220.4, 77.6)
- removed the REF** at (189.6, 34.6)
- removed the REF** at (158.7, 149.2)
- removed the REF** at (220.4, 63.2)
- removed the REF** at (127.9, 163.5)
- removed the REF** at (158.7, 120.5)
- removed the REF** at (127.9, 63.2)
- removed the REF** at (220.4, 106.2)
- removed the REF** at (127.9, 106.2)
Connections:
- R1 pad 2: Board_32-SIG -> Board_32-Net-(U3-Collector)
- R1 pad 2: Board_25-SIG -> Board_25-Net-(U3-Collector)
- R1 pad 2: Board_9-SIG -> Board_9-Net-(U3-Collector)
- R1 pad 2: Board_38-SIG -> Board_38-Net-(U3-Collector)
- R1 pad 2: Board_49-SIG -> Board_49-Net-(U3-Collector)
- R1 pad 2: Board_29-SIG -> Board_29-Net-(U3-Collector)
- R1 pad 2: Board_24-SIG -> Board_24-Net-(U3-Collector)
- R1 pad 2: Board_26-SIG -> Board_26-Net-(U3-Collector)
- R1 pad 2: Board_20-SIG -> Board_20-Net-(U3-Collector)
- R1 pad 2: Board_18-SIG -> Board_18-Net-(U3-Collector)
- R1 pad 2: Board_19-SIG -> Board_19-Net-(U3-Collector)
- R1 pad 2: Board_48-SIG -> Board_48-Net-(U3-Collector)
- R1 pad 2: Board_40-SIG -> Board_40-Net-(U3-Collector)
- R1 pad 2: Board_14-SIG -> Board_14-Net-(U3-Collector)
- R1 pad 2: Board_16-SIG -> Board_16-Net-(U3-Collector)
- R1 pad 2: Board_43-SIG -> Board_43-Net-(U3-Collector)
- R1 pad 2: Board_5-SIG -> Board_5-Net-(U3-Collector)
- R1 pad 2: Board_36-SIG -> Board_36-Net-(U3-Collector)
- R1 pad 2: Board_22-SIG -> Board_22-Net-(U3-Collector)
- R1 pad 2: Board_7-SIG -> Board_7-Net-(U3-Collector)
- R1 pad 2: Board_30-SIG -> Board_30-Net-(U3-Collector)
- R1 pad 2: Board_1-SIG -> Board_1-Net-(U3-Collector)
- R1 pad 2: Board_17-SIG -> Board_17-Net-(U3-Collector)
- R1 pad 2: Board_21-SIG -> Board_21-Net-(U3-Collector)
- R1 pad 2: Board_10-SIG -> Board_10-Net-(U3-Collector)
- R1 pad 2: Board_3-SIG -> Board_3-Net-(U3-Collector)
- R1 pad 2: Board_11-SIG -> Board_11-Net-(U3-Collector)
- R1 pad 2: Board_4-SIG -> Board_4-Net-(U3-Collector)
- R1 pad 2: Board_44-SIG -> Board_44-Net-(U3-Collector)
- R1 pad 2: Board_0-SIG -> Board_0-Net-(U3-Collector)
- R1 pad 2: Board_15-SIG -> Board_15-Net-(U3-Collector)
- R1 pad 2: Board_42-SIG -> Board_42-Net-(U3-Collector)
- R1 pad 2: Board_33-SIG -> Board_33-Net-(U3-Collector)
- R1 pad 2: Board_39-SIG -> Board_39-Net-(U3-Collector)
- R1 pad 2: Board_34-SIG -> Board_34-Net-(U3-Collector)
- R1 pad 2: Board_12-SIG -> Board_12-Net-(U3-Collector)
- R1 pad 2: Board_6-SIG -> Board_6-Net-(U3-Collector)
- R1 pad 2: Board_31-SIG -> Board_31-Net-(U3-Collector)
- R1 pad 2: Board_2-SIG -> Board_2-Net-(U3-Collector)
- R1 pad 2: Board_37-SIG -> Board_37-Net-(U3-Collector)
- R1 pad 2: Board_27-SIG -> Board_27-Net-(U3-Collector)
- R1 pad 2: Board_46-SIG -> Board_46-Net-(U3-Collector)
- R1 pad 2: Board_23-SIG -> Board_23-Net-(U3-Collector)
- R1 pad 2: Board_13-SIG -> Board_13-Net-(U3-Collector)
- R1 pad 2: Board_8-SIG -> Board_8-Net-(U3-Collector)
- R1 pad 2: Board_35-SIG -> Board_35-Net-(U3-Collector)
- R1 pad 2: Board_41-SIG -> Board_41-Net-(U3-Collector)
- R1 pad 2: Board_45-SIG -> Board_45-Net-(U3-Collector)
- R1 pad 2: Board_47-SIG -> Board_47-Net-(U3-Collector)
- R1 pad 2: Board_28-SIG -> Board_28-Net-(U3-Collector)
- R3 pad 1: Board_1-Net-(U3-Emitter) -> Board_1-SIG
- R3 pad 1: Board_33-Net-(U3-Emitter) -> Board_33-SIG
- R3 pad 1: Board_24-Net-(U3-Emitter) -> Board_24-SIG
- R3 pad 1: Board_49-Net-(U3-Emitter) -> Board_49-SIG
- R3 pad 1: Board_34-Net-(U3-Emitter) -> Board_34-SIG
- R3 pad 1: Board_20-Net-(U3-Emitter) -> Board_20-SIG
- R3 pad 1: Board_6-Net-(U3-Emitter) -> Board_6-SIG
- R3 pad 1: Board_48-Net-(U3-Emitter) -> Board_48-SIG
- R3 pad 1: Board_18-Net-(U3-Emitter) -> Board_18-SIG
- R3 pad 1: Board_16-Net-(U3-Emitter) -> Board_16-SIG
- R3 pad 1: Board_7-Net-(U3-Emitter) -> Board_7-SIG
- R3 pad 1: Board_28-Net-(U3-Emitter) -> Board_28-SIG
- R3 pad 1: Board_5-Net-(U3-Emitter) -> Board_5-SIG
- R3 pad 1: Board_40-Net-(U3-Emitter) -> Board_40-SIG
- R3 pad 1: Board_8-Net-(U3-Emitter) -> Board_8-SIG
- R3 pad 1: Board_9-Net-(U3-Emitter) -> Board_9-SIG
- R3 pad 1: Board_10-Net-(U3-Emitter) -> Board_10-SIG
- R3 pad 1: Board_0-Net-(U3-Emitter) -> Board_0-SIG
- R3 pad 1: Board_15-Net-(U3-Emitter) -> Board_15-SIG
- R3 pad 1: Board_11-Net-(U3-Emitter) -> Board_11-SIG
- R3 pad 1: Board_21-Net-(U3-Emitter) -> Board_21-SIG
- R3 pad 1: Board_36-Net-(U3-Emitter) -> Board_36-SIG
- R3 pad 1: Board_32-Net-(U3-Emitter) -> Board_32-SIG
- R3 pad 1: Board_38-Net-(U3-Emitter) -> Board_38-SIG
- R3 pad 1: Board_27-Net-(U3-Emitter) -> Board_27-SIG
- R3 pad 1: Board_43-Net-(U3-Emitter) -> Board_43-SIG
- R3 pad 1: Board_23-Net-(U3-Emitter) -> Board_23-SIG
- R3 pad 1: Board_17-Net-(U3-Emitter) -> Board_17-SIG
- R3 pad 1: Board_30-Net-(U3-Emitter) -> Board_30-SIG
- R3 pad 1: Board_41-Net-(U3-Emitter) -> Board_41-SIG
- R3 pad 1: Board_45-Net-(U3-Emitter) -> Board_45-SIG
- R3 pad 1: Board_29-Net-(U3-Emitter) -> Board_29-SIG
- R3 pad 1: Board_46-Net-(U3-Emitter) -> Board_46-SIG
- R3 pad 1: Board_35-Net-(U3-Emitter) -> Board_35-SIG
- R3 pad 1: Board_14-Net-(U3-Emitter) -> Board_14-SIG
- R3 pad 1: Board_13-Net-(U3-Emitter) -> Board_13-SIG
- R3 pad 1: Board_3-Net-(U3-Emitter) -> Board_3-SIG
- R3 pad 1: Board_42-Net-(U3-Emitter) -> Board_42-SIG
- R3 pad 1: Board_31-Net-(U3-Emitter) -> Board_31-SIG
- R3 pad 1: Board_39-Net-(U3-Emitter) -> Board_39-SIG
- R3 pad 1: Board_4-Net-(U3-Emitter) -> Board_4-SIG
- R3 pad 1: Board_12-Net-(U3-Emitter) -> Board_12-SIG
- R3 pad 1: Board_2-Net-(U3-Emitter) -> Board_2-SIG
- R3 pad 1: Board_22-Net-(U3-Emitter) -> Board_22-SIG
- R3 pad 1: Board_25-Net-(U3-Emitter) -> Board_25-SIG
- R3 pad 1: Board_47-Net-(U3-Emitter) -> Board_47-SIG
- R3 pad 1: Board_19-Net-(U3-Emitter) -> Board_19-SIG
- R3 pad 1: Board_37-Net-(U3-Emitter) -> Board_37-SIG
- R3 pad 1: Board_44-Net-(U3-Emitter) -> Board_44-SIG
- R3 pad 1: Board_26-Net-(U3-Emitter) -> Board_26-SIG
- U3 pad 3: Board_48-SIG -> Board_48-Net-(U3-Collector)
- U3 pad 4: Board_48-Net-(U3-Emitter) -> Board_48-SIG
- U3 pad 3: Board_8-SIG -> Board_8-Net-(U3-Collector)
- U3 pad 4: Board_8-Net-(U3-Emitter) -> Board_8-SIG
- U3 pad 3: Board_49-SIG -> Board_49-Net-(U3-Collector)
- U3 pad 4: Board_49-Net-(U3-Emitter) -> Board_49-SIG
- U3 pad 3: Board_10-SIG -> Board_10-Net-(U3-Collector)
- U3 pad 4: Board_10-Net-(U3-Emitter) -> Board_10-SIG
- U3 pad 3: Board_34-SIG -> Board_34-Net-(U3-Collector)
- U3 pad 4: Board_34-Net-(U3-Emitter) -> Board_34-SIG
- U3 pad 3: Board_33-SIG -> Board_33-Net-(U3-Collector)
- U3 pad 4: Board_33-Net-(U3-Emitter) -> Board_33-SIG
- U3 pad 3: Board_3-SIG -> Board_3-Net-(U3-Collector)
- U3 pad 4: Board_3-Net-(U3-Emitter) -> Board_3-SIG
- U3 pad 3: Board_47-SIG -> Board_47-Net-(U3-Collector)
- U3 pad 4: Board_47-Net-(U3-Emitter) -> Board_47-SIG
- U3 pad 3: Board_12-SIG -> Board_12-Net-(U3-Collector)
- U3 pad 4: Board_12-Net-(U3-Emitter) -> Board_12-SIG
- U3 pad 3: Board_15-SIG -> Board_15-Net-(U3-Collector)
- U3 pad 4: Board_15-Net-(U3-Emitter) -> Board_15-SIG
- U3 pad 3: Board_24-SIG -> Board_24-Net-(U3-Collector)
- U3 pad 4: Board_24-Net-(U3-Emitter) -> Board_24-SIG
- U3 pad 3: Board_16-SIG -> Board_16-Net-(U3-Collector)
- U3 pad 4: Board_16-Net-(U3-Emitter) -> Board_16-SIG
- U3 pad 3: Board_26-SIG -> Board_26-Net-(U3-Collector)
- U3 pad 4: Board_26-Net-(U3-Emitter) -> Board_26-SIG
- U3 pad 3: Board_30-SIG -> Board_30-Net-(U3-Collector)
- U3 pad 4: Board_30-Net-(U3-Emitter) -> Board_30-SIG
- U3 pad 3: Board_20-SIG -> Board_20-Net-(U3-Collector)
- U3 pad 4: Board_20-Net-(U3-Emitter) -> Board_20-SIG
- U3 pad 3: Board_29-SIG -> Board_29-Net-(U3-Collector)
- U3 pad 4: Board_29-Net-(U3-Emitter) -> Board_29-SIG
- U3 pad 3: Board_1-SIG -> Board_1-Net-(U3-Collector)
- U3 pad 4: Board_1-Net-(U3-Emitter) -> Board_1-SIG
- U3 pad 3: Board_14-SIG -> Board_14-Net-(U3-Collector)
- U3 pad 4: Board_14-Net-(U3-Emitter) -> Board_14-SIG
- U3 pad 3: Board_25-SIG -> Board_25-Net-(U3-Collector)
- U3 pad 4: Board_25-Net-(U3-Emitter) -> Board_25-SIG
- U3 pad 3: Board_35-SIG -> Board_35-Net-(U3-Collector)
- U3 pad 4: Board_35-Net-(U3-Emitter) -> Board_35-SIG
- U3 pad 3: Board_11-SIG -> Board_11-Net-(U3-Collector)
- U3 pad 4: Board_11-Net-(U3-Emitter) -> Board_11-SIG
- U3 pad 3: Board_45-SIG -> Board_45-Net-(U3-Collector)
- U3 pad 4: Board_45-Net-(U3-Emitter) -> Board_45-SIG
- U3 pad 3: Board_19-SIG -> Board_19-Net-(U3-Collector)
- U3 pad 4: Board_19-Net-(U3-Emitter) -> Board_19-SIG
- U3 pad 3: Board_2-SIG -> Board_2-Net-(U3-Collector)
- U3 pad 4: Board_2-Net-(U3-Emitter) -> Board_2-SIG
- U3 pad 3: Board_22-SIG -> Board_22-Net-(U3-Collector)
- U3 pad 4: Board_22-Net-(U3-Emitter) -> Board_22-SIG
- U3 pad 3: Board_38-SIG -> Board_38-Net-(U3-Collector)
- U3 pad 4: Board_38-Net-(U3-Emitter) -> Board_38-SIG
- U3 pad 3: Board_7-SIG -> Board_7-Net-(U3-Collector)
- U3 pad 4: Board_7-Net-(U3-Emitter) -> Board_7-SIG
- U3 pad 3: Board_36-SIG -> Board_36-Net-(U3-Collector)
- U3 pad 4: Board_36-Net-(U3-Emitter) -> Board_36-SIG
- U3 pad 3: Board_18-SIG -> Board_18-Net-(U3-Collector)
- U3 pad 4: Board_18-Net-(U3-Emitter) -> Board_18-SIG
- U3 pad 3: Board_5-SIG -> Board_5-Net-(U3-Collector)
- U3 pad 4: Board_5-Net-(U3-Emitter) -> Board_5-SIG
- U3 pad 3: Board_40-SIG -> Board_40-Net-(U3-Collector)
- U3 pad 4: Board_40-Net-(U3-Emitter) -> Board_40-SIG
- U3 pad 3: Board_0-SIG -> Board_0-Net-(U3-Collector)
- U3 pad 4: Board_0-Net-(U3-Emitter) -> Board_0-SIG
- U3 pad 3: Board_41-SIG -> Board_41-Net-(U3-Collector)
- U3 pad 4: Board_41-Net-(U3-Emitter) -> Board_41-SIG
- U3 pad 3: Board_6-SIG -> Board_6-Net-(U3-Collector)
- U3 pad 4: Board_6-Net-(U3-Emitter) -> Board_6-SIG
- U3 pad 3: Board_31-SIG -> Board_31-Net-(U3-Collector)
- U3 pad 4: Board_31-Net-(U3-Emitter) -> Board_31-SIG
- U3 pad 3: Board_23-SIG -> Board_23-Net-(U3-Collector)
- U3 pad 4: Board_23-Net-(U3-Emitter) -> Board_23-SIG
- U3 pad 3: Board_28-SIG -> Board_28-Net-(U3-Collector)
- U3 pad 4: Board_28-Net-(U3-Emitter) -> Board_28-SIG
- U3 pad 3: Board_4-SIG -> Board_4-Net-(U3-Collector)
- U3 pad 4: Board_4-Net-(U3-Emitter) -> Board_4-SIG
- U3 pad 3: Board_21-SIG -> Board_21-Net-(U3-Collector)
- U3 pad 4: Board_21-Net-(U3-Emitter) -> Board_21-SIG
- U3 pad 3: Board_13-SIG -> Board_13-Net-(U3-Collector)
- U3 pad 4: Board_13-Net-(U3-Emitter) -> Board_13-SIG
- U3 pad 3: Board_46-SIG -> Board_46-Net-(U3-Collector)
- U3 pad 4: Board_46-Net-(U3-Emitter) -> Board_46-SIG
- U3 pad 3: Board_27-SIG -> Board_27-Net-(U3-Collector)
- U3 pad 4: Board_27-Net-(U3-Emitter) -> Board_27-SIG
- U3 pad 3: Board_43-SIG -> Board_43-Net-(U3-Collector)
- U3 pad 4: Board_43-Net-(U3-Emitter) -> Board_43-SIG
- U3 pad 3: Board_32-SIG -> Board_32-Net-(U3-Collector)
- U3 pad 4: Board_32-Net-(U3-Emitter) -> Board_32-SIG
- U3 pad 3: Board_42-SIG -> Board_42-Net-(U3-Collector)
- U3 pad 4: Board_42-Net-(U3-Emitter) -> Board_42-SIG
- U3 pad 3: Board_9-SIG -> Board_9-Net-(U3-Collector)
- U3 pad 4: Board_9-Net-(U3-Emitter) -> Board_9-SIG
- U3 pad 3: Board_37-SIG -> Board_37-Net-(U3-Collector)
- U3 pad 4: Board_37-Net-(U3-Emitter) -> Board_37-SIG
- U3 pad 3: Board_39-SIG -> Board_39-Net-(U3-Collector)
- U3 pad 4: Board_39-Net-(U3-Emitter) -> Board_39-SIG
- U3 pad 3: Board_44-SIG -> Board_44-Net-(U3-Collector)
- U3 pad 4: Board_44-Net-(U3-Emitter) -> Board_44-SIG
- U3 pad 3: Board_17-SIG -> Board_17-Net-(U3-Collector)
- U3 pad 4: Board_17-Net-(U3-Emitter) -> Board_17-SIG
Routing:
- net Board_8-Net-(U3-Emitter): track 7.64 -> 0.00 mm
- net Board_48-Net-(U3-Emitter): track 7.64 -> 0.00 mm
- net Board_38-Net-(U3-Emitter): track 7.64 -> 0.00 mm
- net Board_28-Net-(U3-Emitter): track 7.64 -> 0.00 mm
- net Board_23-Net-(U3-Emitter): track 7.64 -> 0.00 mm
- net Board_18-Net-(U3-Emitter): track 7.64 -> 0.00 mm
- net Board_13-Net-(U3-Emitter): track 7.64 -> 0.00 mm
- net Board_3-Net-(U3-Emitter): track 7.64 -> 0.00 mm
- net Board_6-Net-(U3-Emitter): track 7.64 -> 0.00 mm
- net Board_46-Net-(U3-Emitter): track 7.64 -> 0.00 mm
- net Board_36-Net-(U3-Emitter): track 7.64 -> 0.00 mm
- net Board_33-Net-(U3-Emitter): track 7.64 -> 0.00 mm
- net Board_26-Net-(U3-Emitter): track 7.64 -> 0.00 mm
- net Board_21-Net-(U3-Emitter): track 7.64 -> 0.00 mm
- net Board_16-Net-(U3-Emitter): track 7.64 -> 0.00 mm
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